File: PCB/Knomberpad.sch (KiCad schematic (older format))
At the start: 38 parts, among them SW1 Rotary_Encoder, U1 ProMicro

Commit message: Change footprints
Parts:
- added D19: D_Small, keebio:Diode, symbol Device:D_Small
- D1, D12, D13, D14, D2, D3, D4, D5, D6, D7: footprint ai03:D_SOD-123-Pretty -> keebio:Diode
- D10: renamed from D9; footprint ai03:D_SOD-123-Pretty -> keebio:Diode
- D11: renamed from D10; footprint ai03:D_SOD-123-Pretty -> keebio:Diode
- D15: renamed from D18; footprint ai03:D_SOD-123-Pretty -> keebio:Diode
- D16: renamed from D15; footprint ai03:D_SOD-123-Pretty -> keebio:Diode
- D17: renamed from D16; footprint ai03:D_SOD-123-Pretty -> keebio:Diode
- D18: renamed from D17; footprint ai03:D_SOD-123-Pretty -> keebio:Diode
- D8: renamed from D11; footprint ai03:D_SOD-123-Pretty -> keebio:Diode
- D9: renamed from D8; footprint ai03:D_SOD-123-Pretty -> keebio:Diode
- MX15: renamed from MX18; footprint ai03_switch:MX-2U -> ai03_switch:MX-2U-NoLED
- SW19: renamed from SW1; value Rotary_Encoder -> RT1; symbol Device:Rotary_Encoder -> Device:Rotary_Encoder_Switch
- renumbered MX9 to MX10, MX10 to MX11, MX15 to MX16, MX16 to MX17, MX17 to MX18, MX11 to MX8, MX8 to MX9
Connections:
- net COL0: now also U1.20 (A3/PF4); no longer U1.16 (15/PB1)
- net COL1: now also U1.19 (A2/PF5); no longer U1.17 (A0/PF7)
- net COL2: now also U1.16 (15/PB1); no longer U1.18 (A1/PF6)
- net COL3: now also SW19.S2, U1.17 (A0/PF7); no longer U1.19 (A2/PF5)
- net ROT_A: now also U1.6 (3/PD0); no longer U1.14 (16/PB2)
- net ROT_B: now also U1.7 (4/PD4); no longer U1.5 (2/PD1)
- net ROT_C: now also U1.23 (GND); no longer U1.4 (GND)
- net ROW0: now also U1.18 (A1/PF6); no longer U1.20 (A3/PF4)
- net ROW1: now also D8.1 (K), U1.15 (14/PB3); no longer U1.13 (10/PB6)
- net ROW2: now also U1.14 (16/PB2); no longer D8.1 (K), U1.10 (7/PE6)
- net ROW3: now also D15.1 (K), U1.13 (10/PB6); no longer U1.11 (8/PB4)
- net ROW4: now also U1.5 (2/PD1), D19.1 (K); no longer D15.1 (K), U1.12 (9/PB5)
- new net: D19.2 (A), SW19.S1
Other:
- moved on the sheet: D15, D8, MX15, MX8
